Commit message: made changes

File: nuturtle_description/urdf/turtlebot3_burger.urdf.xacro (robot description, xacro)
@@ -8,11 +8,11 @@
 <xacro:property name="track_width" value = "${params['track_width']}" />
 <xacro:arg name="color" default="black" />
-  <link name="$(arg color)_base_footprint"/>
-  <joint name="$(arg color)_base_joint" type="fixed">
-    <parent link="$(arg color)_base_footprint"/>
-    <child link="$(arg color)_base_link"/>
+  <link name="$(arg color):base_footprint"/>
+  <joint name="$(arg color):base_joint" type="fixed">
+    <parent link="$(arg color):base_footprint"/>
+    <child link="$(arg color):base_link"/>
     <origin xyz="0.0 0.0 0.010" rpy="0 0 0"/>
   </joint>
-  <link name="$(arg color)_base_link">
+  <link name="$(arg color):base_link">
     <visual>light_black
       <origin xyz="-0.032 0 0.0" rpy="0 0 0"/>
@@ -36,11 +36,11 @@
     </inertial>
   </link>
-  <joint name="$(arg color)_wheel_left_joint" type="continuous">
-    <parent link="$(arg color)_base_link"/>
-    <child link="$(arg color)_wheel_left_link"/>
+  <joint name="$(arg color):wheel_left_joint" type="continuous">
+    <parent link="$(arg color):base_link"/>
+    <child link="$(arg color):wheel_left_link"/>
     <origin xyz="0.0 ${track_width/2} 0.023" rpy="-1.57 0 0"/>
     <axis xyz="0 0 1"/>
   </joint>
-  <link name="$(arg color)_wheel_left_link">
+  <link name="$(arg color):wheel_left_link">
     <visual>
       <origin xyz="0 0 0" rpy="1.57 0 0"/>
@@ -64,11 +64,11 @@
       </inertial>
   </link>
-  <joint name="$(arg color)_wheel_right_joint" type="continuous">
-    <parent link="$(arg color)_base_link"/>
-    <child link="$(arg color)_wheel_right_link"/>
+  <joint name="$(arg color):wheel_right_joint" type="continuous">
+    <parent link="$(arg color):base_link"/>
+    <child link="$(arg color):wheel_right_link"/>
     <origin xyz="0.0 -${track_width/2} 0.023" rpy="-1.57 0 0"/>
     <axis xyz="0 0 1"/>
   </joint>
-  <link name="$(arg color)_wheel_right_link">
+  <link name="$(arg color):wheel_right_link">
     <visual>
       <origin xyz="0 0 0" rpy="1.57 0 0"/>
@@ -92,10 +92,10 @@
       </inertial>
   </link>
-  <joint name="$(arg color)_caster_back_joint" type="fixed">
-    <parent link="$(arg color)_base_link"/>
-    <child link="$(arg color)_caster_back_link"/>
+  <joint name="$(arg color):caster_back_joint" type="fixed">
+    <parent link="$(arg color):base_link"/>
+    <child link="$(arg color):caster_back_link"/>
     <origin xyz="-0.081 0 -0.004" rpy="-1.57 0 0"/>
   </joint>
-  <link name="$(arg color)_caster_back_link">
+  <link name="$(arg color):caster_back_link">
     <collision>
       <origin xyz="0 0.001 0" rpy="0 0 0"/>
@@ -112,16 +112,16 @@
     </inertial>
   </link>
-  <joint name="$(arg color)_imu_joint" type="fixed">
-    <parent link="$(arg color)_base_link"/>
-    <child link="$(arg color)_imu_link"/>
+  <joint name="$(arg color):imu_joint" type="fixed">
+    <parent link="$(arg color):base_link"/>
+    <child link="$(arg color):imu_link"/>
     <origin xyz="-0.032 0 0.068" rpy="0 0 0"/>
   </joint>
-  <link name="$(arg color)_imu_link"/>
-  <joint name="$(arg color)_scan_joint" type="fixed">
-    <parent link="$(arg color)_base_link"/>
-    <child link="$(arg color)_base_scan"/>
+  <link name="$(arg color):imu_link"/>
+  <joint name="$(arg color):scan_joint" type="fixed">
+    <parent link="$(arg color):base_link"/>
+    <child link="$(arg color):base_scan"/>
     <origin xyz="-0.032 0 0.172" rpy="0 0 0"/>
   </joint>
-  <link name="$(arg color)_base_scan">
+  <link name="$(arg color):base_scan">
     <visual>
       <origin xyz="0 0 0.0" rpy="0 0 0"/>

Commit message: removed ':' with '_'

File: nuturtle_description/urdf/turtlebot3_burger.urdf.xacro (robot description, xacro)
@@ -8,11 +8,11 @@
 <xacro:property name="track_width" value = "${params['track_width']}" />
 <xacro:arg name="color" default="black" />
-  <link name="$(arg color):base_footprint"/>
-  <joint name="$(arg color):base_joint" type="fixed">
-    <parent link="$(arg color):base_footprint"/>
-    <child link="$(arg color):base_link"/>
+  <link name="$(arg color)_base_footprint"/>
+  <joint name="$(arg color)_base_joint" type="fixed">
+    <parent link="$(arg color)_base_footprint"/>
+    <child link="$(arg color)_base_link"/>
     <origin xyz="0.0 0.0 0.010" rpy="0 0 0"/>
   </joint>
-  <link name="$(arg color):base_link">
+  <link name="$(arg color)_base_link">
     <visual>light_black
       <origin xyz="-0.032 0 0.0" rpy="0 0 0"/>
@@ -36,11 +36,11 @@
     </inertial>
   </link>
-  <joint name="$(arg color):wheel_left_joint" type="continuous">
-    <parent link="$(arg color):base_link"/>
-    <child link="$(arg color):wheel_left_link"/>
+  <joint name="$(arg color)_wheel_left_joint" type="continuous">
+    <parent link="$(arg color)_base_link"/>
+    <child link="$(arg color)_wheel_left_link"/>
     <origin xyz="0.0 ${track_width/2} 0.023" rpy="-1.57 0 0"/>
     <axis xyz="0 0 1"/>
   </joint>
-  <link name="$(arg color):wheel_left_link">
+  <link name="$(arg color)_wheel_left_link">
     <visual>
       <origin xyz="0 0 0" rpy="1.57 0 0"/>
@@ -64,11 +64,11 @@
       </inertial>
   </link>
-  <joint name="$(arg color):wheel_right_joint" type="continuous">
-    <parent link="$(arg color):base_link"/>
-    <child link="$(arg color):wheel_right_link"/>
+  <joint name="$(arg color)_wheel_right_joint" type="continuous">
+    <parent link="$(arg color)_base_link"/>
+    <child link="$(arg color)_wheel_right_link"/>
     <origin xyz="0.0 -${track_width/2} 0.023" rpy="-1.57 0 0"/>
     <axis xyz="0 0 1"/>
   </joint>
-  <link name="$(arg color):wheel_right_link">
+  <link name="$(arg color)_wheel_right_link">
     <visual>
       <origin xyz="0 0 0" rpy="1.57 0 0"/>
@@ -92,10 +92,10 @@
       </inertial>
   </link>
-  <joint name="$(arg color):caster_back_joint" type="fixed">
-    <parent link="$(arg color):base_link"/>
-    <child link="$(arg color):caster_back_link"/>
+  <joint name="$(arg color)_caster_back_joint" type="fixed">
+    <parent link="$(arg color)_base_link"/>
+    <child link="$(arg color)_caster_back_link"/>
     <origin xyz="-0.081 0 -0.004" rpy="-1.57 0 0"/>
   </joint>
-  <link name="$(arg color):caster_back_link">
+  <link name="$(arg color)_caster_back_link">
     <collision>
       <origin xyz="0 0.001 0" rpy="0 0 0"/>
@@ -112,16 +112,16 @@
     </inertial>
   </link>
-  <joint name="$(arg color):imu_joint" type="fixed">
-    <parent link="$(arg color):base_link"/>
-    <child link="$(arg color):imu_link"/>
+  <joint name="$(arg color)_imu_joint" type="fixed">
+    <parent link="$(arg color)_base_link"/>
+    <child link="$(arg color)_imu_link"/>
     <origin xyz="-0.032 0 0.068" rpy="0 0 0"/>
   </joint>
-  <link name="$(arg color):imu_link"/>
-  <joint name="$(arg color):scan_joint" type="fixed">
-    <parent link="$(arg color):base_link"/>
-    <child link="$(arg color):base_scan"/>
+  <link name="$(arg color)_imu_link"/>
+  <joint name="$(arg color)_scan_joint" type="fixed">
+    <parent link="$(arg color)_base_link"/>
+    <child link="$(arg color)_base_scan"/>
     <origin xyz="-0.032 0 0.172" rpy="0 0 0"/>
   </joint>
-  <link name="$(arg color):base_scan">
+  <link name="$(arg color)_base_scan">
     <visual>
       <origin xyz="0 0 0.0" rpy="0 0 0"/>

Commit message: replaced '_' with '-'

File: nuturtle_description/urdf/turtlebot3_burger.urdf.xacro (robot description, xacro)
@@ -2,5 +2,4 @@
 <robot name="turtlebot3_burger" xmlns:xacro="http://ros.org/wiki/xacro">
 <xacro:include filename="$(find nuturtle_description)/urdf/common_properties.xacro"/>
-<!-- <xacro:include filename="$(find turtlebot3_description)/urdf/turtlebot3_burger.gazebo.xacro"/> -->
 <xacro:property name="diff_yaml" value="$(find nuturtle_description)/config/diff_params.yaml"/>
 <xacro:property name="params" value = "${xacro.load_yaml(diff_yaml)}"/>
@@ -8,11 +7,11 @@
 <xacro:property name="track_width" value = "${params['track_width']}" />
 <xacro:arg name="color" default="black" />
-  <link name="$(arg color)_base_footprint"/>
-  <joint name="$(arg color)_base_joint" type="fixed">
-    <parent link="$(arg color)_base_footprint"/>
-    <child link="$(arg color)_base_link"/>
+  <link name="$(arg color)-base_footprint"/>
+  <joint name="$(arg color)-base_joint" type="fixed">
+    <parent link="$(arg color)-base_footprint"/>
+    <child link="$(arg color)-base_link"/>
     <origin xyz="0.0 0.0 0.010" rpy="0 0 0"/>
   </joint>
-  <link name="$(arg color)_base_link">
+  <link name="$(arg color)-base_link">
     <visual>light_black
       <origin xyz="-0.032 0 0.0" rpy="0 0 0"/>
@@ -36,11 +35,11 @@
     </inertial>
   </link>
-  <joint name="$(arg color)_wheel_left_joint" type="continuous">
-    <parent link="$(arg color)_base_link"/>
-    <child link="$(arg color)_wheel_left_link"/>
+  <joint name="$(arg color)-wheel_left_joint" type="continuous">
+    <parent link="$(arg color)-base_link"/>
+    <child link="$(arg color)-wheel_left_link"/>
     <origin xyz="0.0 ${track_width/2} 0.023" rpy="-1.57 0 0"/>
     <axis xyz="0 0 1"/>
   </joint>
-  <link name="$(arg color)_wheel_left_link">
+  <link name="$(arg color)-wheel_left_link">
     <visual>
       <origin xyz="0 0 0" rpy="1.57 0 0"/>
@@ -64,11 +63,11 @@
       </inertial>
   </link>
-  <joint name="$(arg color)_wheel_right_joint" type="continuous">
-    <parent link="$(arg color)_base_link"/>
-    <child link="$(arg color)_wheel_right_link"/>
+  <joint name="$(arg color)-wheel_right_joint" type="continuous">
+    <parent link="$(arg color)-base_link"/>
+    <child link="$(arg color)-wheel_right_link"/>
     <origin xyz="0.0 -${track_width/2} 0.023" rpy="-1.57 0 0"/>
     <axis xyz="0 0 1"/>
   </joint>
-  <link name="$(arg color)_wheel_right_link">
+  <link name="$(arg color)-wheel_right_link">
     <visual>
       <origin xyz="0 0 0" rpy="1.57 0 0"/>
@@ -92,10 +91,10 @@
       </inertial>
   </link>
-  <joint name="$(arg color)_caster_back_joint" type="fixed">
-    <parent link="$(arg color)_base_link"/>
-    <child link="$(arg color)_caster_back_link"/>
+  <joint name="$(arg color)-caster_back_joint" type="fixed">
+    <parent link="$(arg color)-base_link"/>
+    <child link="$(arg color)-caster_back_link"/>
     <origin xyz="-0.081 0 -0.004" rpy="-1.57 0 0"/>
   </joint>
-  <link name="$(arg color)_caster_back_link">
+  <link name="$(arg color)-caster_back_link">
     <collision>
       <origin xyz="0 0.001 0" rpy="0 0 0"/>
@@ -112,16 +111,16 @@
     </inertial>
   </link>
-  <joint name="$(arg color)_imu_joint" type="fixed">
-    <parent link="$(arg color)_base_link"/>
-    <child link="$(arg color)_imu_link"/>
+  <joint name="$(arg color)-imu_joint" type="fixed">
+    <parent link="$(arg color)-base_link"/>
+    <child link="$(arg color)-imu_link"/>
     <origin xyz="-0.032 0 0.068" rpy="0 0 0"/>
   </joint>
-  <link name="$(arg color)_imu_link"/>
-  <joint name="$(arg color)_scan_joint" type="fixed">
-    <parent link="$(arg color)_base_link"/>
-    <child link="$(arg color)_base_scan"/>
+  <link name="$(arg color)-imu_link"/>
+  <joint name="$(arg color)-scan_joint" type="fixed">
+    <parent link="$(arg color)-base_link"/>
+    <child link="$(arg color)-base_scan"/>
     <origin xyz="-0.032 0 0.172" rpy="0 0 0"/>
   </joint>
-  <link name="$(arg color)_base_scan">
+  <link name="$(arg color)-base_scan">
     <visual>
       <origin xyz="0 0 0.0" rpy="0 0 0"/>

Commit message: added ability to change collision of the base link

File: nuturtle_description/urdf/turtlebot3_burger.urdf.xacro (robot description, xacro)
@@ -6,4 +6,5 @@
 <xacro:property name="wheel_radius" value = "${params['wheel_radius']}" />
 <xacro:property name="track_width" value = "${params['track_width']}" />
+<xacro:property name="collision_radius" value = "${params['collision_radius']}" />
 <xacro:arg name="color" default="black" />
   <link name="$(arg color)-base_footprint"/>
@@ -24,5 +25,11 @@
       <origin xyz="-0.032 0 0.070" rpy="0 0 0"/>
       <geometry>
-        <box size="0.140 0.140 0.143"/>
+          <!-- <cylinder length="0.143" radius="${collision_radius}"/> -->
+        <xacro:if value="${collision_radius == 0.0}">
+          <box size="0.140 0.140 0.143"/>
+        </xacro:if>
+        <xacro:if value="${collision_radius != 0.0}">
+          <cylinder length="0.143" radius="${collision_radius}"/>
+        </xacro:if>
       </geometry>
     </collision>

Commit message: working on laser scan

File: nuturtle_description/urdf/turtlebot3_burger.urdf.xacro (robot description, xacro)
@@ -23,5 +23,5 @@
     </visual>
     <collision>
-      <origin xyz="-0.032 0 0.070" rpy="0 0 0"/>
+      <origin xyz="-0.0 0 0.070" rpy="0 0 0"/>
       <geometry>
           <!-- <cylinder length="0.143" radius="${collision_radius}"/> -->
